File: Electronics/PCB_Layout/Resp2.kicad_pcb (KiCad board)
At the start: 2 copper layers, 110.5 x 63.5 mm, 84 parts, among them J1 * POWER12V *, J2 DISPLAY, J3 PWM_EXTN, J4 MOTOR, J5 POS1_SNS, J6 POS2_SNS, J7 KNOB, J8 LED, J9 SWITCH, U1 LM2937xMP, U2 DRV8842PWP, U3 74HC14, U4 NE555

Commit message: updated layout file
Parts:
- added G***: LOGO, Resp2:logo, B.Cu at (60.5, 52.1)
- moved R21 8.25 mm to (61.8, 67.3)
- moved R12 7.30 mm to (46.7, 69.8)
- moved R13 5.75 mm to (41.0, 19.1)
- moved C8 5.12 mm to (20.3, 27.1), turned to 270 degrees
- moved R18 5.08 mm to (54.9, 67.3)
- moved R11 4.59 mm to (20.3, 22.5), turned to 90 degrees
- moved C13 2.96 mm to (38.1, 22.5), turned to 270 degrees
- moved R20 2.80 mm to (41.3, 22.5), turned to 270 degrees
- moved R1 2.66 mm to (40.4, 69.8)
- moved D4 1.45 mm to (46.7, 73.7), turned to 0 degrees
- moved D3 1.35 mm to (40.4, 73.7), turned to 180 degrees
- moved D5 1.05 mm to (46.7, 15.2), turned to 180 degrees
- moved C9 0.54 mm to (46.4, 30.0), turned to 270 degrees
- moved C10 0.46 mm to (34.9, 22.5), turned to 90 degrees
- moved C12 0.46 mm to (23.5, 22.5), turned to 90 degrees
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Routing:
- net GND: track 93.3 -> 103.3 mm, vias 51 -> 61
- net Net-(J8-Pad3): track 16.5 -> 9.25 mm
- net +12V: track 72.7 -> 79.2 mm, vias 13 -> 14
- net Net-(D4-Pad2): track 9.23 -> 4.66 mm
- net Net-(D5-Pad2): track 12.5 -> 8.26 mm
- net /out2: track 36.6 -> 33.0 mm
- net Net-(R14-Pad2): track 32.7 -> 36.3 mm
- net /out1: track 43.9 -> 40.6 mm, vias 3 -> 6
- net Net-(J8-Pad4): track 9.68 -> 6.52 mm
- net /Arduino_motor_ctrl1: track 123.0 -> 125.8 mm, vias 2 -> 1
- net /Arduino_motor_ctrl2: track 115.0 -> 117.8 mm
- net /Arduino_motor_reset: track 119.6 -> 116.9 mm, vias 2 -> 1
- net Net-(C13-Pad2): track 14.0 -> 12.0 mm
- net /Arduino_ok_led: track 28.4 -> 26.9 mm
- net Net-(R24-Pad2): track 23.3 -> 21.9 mm
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Other:
- net class Default: clearance 0.2 -> 0.25
- net class Narrow removed
- rule trace_clearance: 0.2 -> 0.25
- rule trace_min: 0.2 -> 0.25
- board text added: "+ 12V"
- board text added: "+ 5V"
- board text added: "Motor + +"
- board text removed: "+12V"
- board text removed: "+5V"
- board text removed: "Motor +"
